Commit message: feat: Fix deployment, Map subset-controlling policies onto the robot's full joint set
Add a JointAdapter that bridges a policy trained on a subset of joints
(e.g. single arm + hand) with the robot's full command vector
[dual_arm, left_ee, right_ee], using joint names as the source of truth.
Uncontrolled joints are frozen at the live rest pose via set_defaults()
instead of requiring recorded actions. Wired into both eval_g1.py and
eval_g1_sim.py for state gathering, action scattering, and data saving;
make_robot.py now exposes the canonical full_joint_names layout derived
from ROBOT_CONFIGS.

Also:
- Pin DDS to the robot NIC up front in setup_robot_interface; the Unitree
  SDK ignores CYCLONEDDS_URI and otherwise auto-selects the wrong
  interface, so rt/lowstate never arrives. Add net_interface/image_host
  config fields.
- Register third-party lerobot_policy_* plugins before parsing and update
  get_safe_torch_device import to its new module path.
- Switch head camera observation to a single cam_head frame.
- Add an OOM guard (currently disabled) that caps conversion workers to
  fit available RAM in convert_unitree_json_to_lerobot_multi.py.
- Zero the dex3 thumb_0 joint limits in the hand URDFs and disable the
  cv2 preview windows in the image client.

File: unitree_lerobot/eval_robot/assets/unitree_hand/unitree_dex3_left.urdf (robot description, URDF)
Before this commit: robot dex3_left, 15 links, 14 joints
Joints:
- joint left_hand_thumb_0_joint: limit lower=-1.04719755 upper=1.04719755 effort=2.45 velocity=6.857 -> lower=0.0 upper=0.0 effort=2.45 velocity=6.857

File: unitree_lerobot/eval_robot/assets/unitree_hand/unitree_dex3_right.urdf (robot description, URDF)
Before this commit: robot dex3_right, 15 links, 14 joints
Joints:
- joint right_hand_thumb_0_joint: limit lower=-1.04719755 upper=1.04719755 effort=2.45 velocity=6.857 -> lower=0.0 upper=0.0 effort=2.45 velocity=6.857
